File: pcb/33120a.kicad_sch (KiCad schematic)
At the start: 104 parts, among them J1 10 MHz input, J2 10 MHz output, P2 40 MHz output, T101 Transformer_1P_1S, U101 LM361M, U102 74LS132, U103 74HC02, U104 74HC86, U105 74HC74, U106 4066, U107 TL074, U108 L78L12_SOT89, U109 L79L12_SOT89, U110 OCXO, U112 NB3N502

Commit message: added info
Parts:
- CR108: value SZESD9B5.0ST5G -> SMCJ43CA
- T101: value Transformer_1P_1S -> TC1-1T+
Other:
- moved on the sheet: C101, C102, C103, C104, C105, C106, C107, C108, C109, C110, C111, C112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
