File: pcb/33120a.kicad_pcb (KiCad board)
At the start: 2 copper layers, 79.8 x 51.3 mm, 104 parts, among them J1 10 MHz input, J2 10 MHz output, P2 40 MHz output, T101 Transformer_1P_1S, U101 LM361M, U102 74LS132, U103 74HC02, U104 74HC86, U105 74HC74, U106 4066, U107 TL074, U108 L78L12_SOT89, U109 L79L12_SOT89, U110 OCXO, U112 NB3N502

Commit message: silkscreen update
Other:
- board text added: "JLCJLCJLCJLC"
